File: circuit/Eagle/BatNode/BatNode.brd (EAGLE design)
At the start: 99.7 x 48.6 mm, 90 parts, among them IC1 TL974, IC2 TL972, Q1 BC547, U1 ATMEGA328P_PDIP, U3 TPS79147

Commit message: BatNode v0.21
Parts:
- removed C27: 0.1u, SparkFun-Capacitors:0805
- removed IC2: TL972, SparkFun-AnalogIC:SO08
- removed PRG, SDCARD: (no value), SparkFun-Connectors:1X06_LOCK
- removed RTC: (no value), SparkFun-Connectors:1X04_LOCK
- removed U$1: LMV331, BatNodeParts:SOT23-5
- removed U$14, U$2: SPU0410LR5H, BatNodeParts:SPU0410LR5H
- added C19: 22p, SparkFun-Capacitors:CAP-PTH-SMALL
- added JP10, JP11: VOUT, SparkFun-Connectors:1X02_LOCK
- added JP9: VIN, SparkFun-Connectors:1X02_LOCK
- added U4, U5: SPU0410LR5H, BatNodeParts:SPU0410LR5H
- added U6: ATMEGA328P_PDIP, SparkFun-DigitalIC:DIL28-3
- added U7: TPS79147, SparkFun-PowerIC:SOT23-5
- C1: value 22p -> 100u; device SparkFun-Capacitors:CAP-PTH-SMALL -> SparkFun-Capacitors:CPOL-RADIAL-100UF-25V
- C10: value 0.1u -> 680p; device SparkFun-Capacitors:0805 -> resistor:C025-030X050
- C11: value 0.1u -> 1n; device SparkFun-Capacitors:0805 -> resistor:C025-030X050
- C12: device SparkFun-Capacitors:0805 -> resistor:C025-030X050
- C13: value 100n -> 4.7n; device SparkFun-Passives:0805 -> resistor:C025-030X050
- C14: value 100n -> 10n; device SparkFun-Passives:0805 -> resistor:C025-030X050
- C15: value 100n -> 0.1u; device SparkFun-Passives:0805 -> SparkFun-Capacitors:0805
- C16, C17: value 1u -> 100n; device resistor:C025-030X050 -> SparkFun-Passives:0805
- C18: value 0.1u -> 22p; device SparkFun-Capacitors:0805 -> SparkFun-Capacitors:CAP-PTH-SMALL
- C2: value 1u -> 10n; device SparkFun-Capacitors:0805 -> resistor:C025-030X050
- C20: value 4.7n -> 100n; device resistor:C025-030X050 -> SparkFun-Passives:0805
- C21: value 10p -> 0.1u; device resistor:C025-030X050 -> SparkFun-Capacitors:0805
- C22: value 10n -> 1u
- C23: value 0.1u -> 1u; device SparkFun-Capacitors:0805 -> resistor:C025-030X050
- C24: value 1u -> 0.1u; device resistor:C025-030X050 -> SparkFun-Capacitors:0805
- C3, C6: value 10n -> 0.1u; device resistor:C025-030X050 -> SparkFun-Capacitors:0805
- C4: value 100u -> 10p; device SparkFun-Capacitors:CPOL-RADIAL-100UF-25V -> resistor:C025-030X050
- C5: value 22p -> 1u; device SparkFun-Capacitors:CAP-PTH-SMALL -> SparkFun-Capacitors:0805
- C7: value 1n -> 10n
- C8: value 680p -> 1u; device resistor:C025-030X050 -> SparkFun-Capacitors:0805
- IC1: value TL974 -> TL972; device SparkFun-AnalogIC:SO014 -> SparkFun-AnalogIC:SO08
- JP1: value MIC -> PWR; device SparkFun-Connectors:1X03_LOCK -> SparkFun-Connectors:1X02_LOCK
- JP2: value PWR -> MIC; device SparkFun-Connectors:1X02_LOCK -> SparkFun-Connectors:1X04
- JP3: device SparkFun-Connectors:1X04 -> SparkFun-Connectors:1X03_LOCK
- JP5: value BAT -> (none); device SparkFun-Connectors:1X02_LOCK -> SparkFun-Connectors:1X04_LOCK
- JP6, JP7: value VOUT -> (none); device SparkFun-Connectors:1X02_LOCK -> SparkFun-Connectors:1X06_LOCK
- JP8: value VIN -> BAT
- R1: value 4.7k -> 2.2k
- R10: value 2.2k -> PHOTOCELLPTH; device SparkFun-Resistors:AXIAL-0.3 -> SparkFun-Sensors:PHOTOCELL
- R11: value 10k -> 6.8k; device SparkFun-Resistors:AXIAL-0.3 -> SparkFun-Passives:AXIAL-0.3
- R12: value 1k -> 100k
- R13: value 6.8k -> 4.7k
- R14: value 1k -> 10k
- R15: value 6.8k -> 22k
- R18: value 100k -> 22k
- R19: value 100k -> 4.7k
- R2: value 1Meg -> 1k
- R20: value 22k -> 4.7k
- R21: value PHOTOCELLPTH -> 330; device SparkFun-Sensors:PHOTOCELL -> SparkFun-Passives:AXIAL-0.3
- R22: value 330 -> 22k
- R23: value 4.7k -> 22k
- R24: value 22k -> 1k
- R25: value 4.7k -> 10uH
- R26, R28: value 22k -> 220; device SparkFun-Passives:AXIAL-0.3 -> SparkFun-Resistors:AXIAL-0.3
- R27: value 4.7k -> 220; device SparkFun-Passives:AXIAL-0.3 -> SparkFun-Resistors:AXIAL-0.3
- R29: value 1k -> 2.2k; device SparkFun-Passives:AXIAL-0.3 -> SparkFun-Resistors:AXIAL-0.3
- R3: value 47k -> 6.8k
- R30: value 10uH -> 10k; device SparkFun-Passives:AXIAL-0.3 -> SparkFun-Resistors:AXIAL-0.3
- R4: value 47k -> 4.7k
- R5: value 2.2k -> 1Meg
- R6, R7: value 220 -> 47k; device SparkFun-Resistors:AXIAL-0.3 -> SparkFun-Passives:AXIAL-0.3
- R8: value 220 -> 100k; device SparkFun-Resistors:AXIAL-0.3 -> SparkFun-Passives:AXIAL-0.3
- R9: value 10k -> 1k
- U1: value ATMEGA328P_PDIP -> (none); device SparkFun-DigitalIC:DIL28-3 -> SparkFun-Sensors:TO-92
- U2: value (none) -> LMV331; device SparkFun-Sensors:TO-92 -> BatNodeParts:SOT23-5
- U3: value TPS79147 -> LMV324; device SparkFun-PowerIC:SOT23-5 -> SparkFun-AnalogIC:SO014
- moved JP1 99.4 mm to (2.22, 19.4), turned to 270 degrees
- moved JP3 96.4 mm to (98.3, 46.8), turned to 180 degrees
- moved JP8 94.8 mm to (1.59, 3.49), turned to 90 degrees
- moved C21 92.8 mm to (94.6, 5.46)
- moved C25 87.4 mm to (95.2, 14.0)
- moved C23 86.6 mm to (7.94, 7.49)
- moved C17 79.0 mm to (83.8, 32.1)
- moved JP5 77.1 mm to (65.4, 46.7), turned to 180 degrees
- moved C24 76.4 mm to (97.0, 8.89), turned to 270 degrees
- moved U3 76.2 mm to (22.2, 34.0), turned to 270 degrees
- moved R25 69.9 mm to (78.7, 30.2), turned to 270 degrees
- moved JP7 57.8 mm to (87.0, 5.08), turned to 90 degrees
- moved C15 56.8 mm to (29.2, 16.5)
- moved C5 54.0 mm to (16.5, 37.8)
- moved C1 53.8 mm to (6.99, 23.8)
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- renumbered GND-CONNECT to X12, RST to S3, U$15 to U8, V-CONNECT to X11
Connections:
- net A0: now also C14.1, R24.P$2, U6.23; no longer C22.1, R29.P$2, U1.23
- net A1: now also U1.2, U6.24; no longer U1.24, U2.2
- net A2: now also R10.2, R14.P$1, U6.25; no longer R21.2, R9.P$1, U1.25
- net A3: now also U6.26; no longer U1.26
- net AGND: now also C1.2, C12.1, C14.2, C15.2, C3.2, C5.2, C6.2, C8.2, IC1.4, JP1.1, R14.P$2, R22.P$1, R7.P$2, U1.3, U2.2, U3.11; no longer C10.2, C11.2, C12.2, C17.1, C18.2, C2.2, C22.2, C4.2, IC1.11, IC2.4, JP3.1, R26.P$1, R4.P$2, R9.P$2, U$1.2, U2.3
- net CS: now also JP7.6, U6.16; no longer SDCARD.6, U1.16
- net D2: now also U6.4; no longer U1.4
- net D3: now also R26.P$2, U6.5; no longer R6.P$2, U1.5
- net D4: now also U6.6; no longer U1.6
- net D5: now also C4.1, R4.P$2, R5.P$2, U2.4, U6.11; no longer C21.1, R1.P$2, R2.P$2, U$1.4, U1.11
- net D6: now also R27.P$2, U6.12; no longer R7.P$2, U1.12
- net D7: now also R29.P$2, U6.13; no longer R10.P$2, U1.13
- net D8: now also U6.14; no longer U1.14
- net D9: now also R28.P$2, U6.15; no longer R8.P$2, U1.15
- net FILTER: now also C13.2, R13.P$1, R21.P$2, U2.3; no longer C20.2, R22.P$2, R23.P$1, U$1.3
- net GND: now also C16.2, C18.1, C19.1, C20.2, JP5.1, JP6.1, U6.22, U6.8; no longer C1.1, C13.2, C14.2, C5.1, PRG.1, RTC.1, U1.22, U1.8
- net GNDBATT: now also C22.2, C23.2, JP11.2, JP8.1; no longer C24.2, C25.2, JP5.1, JP7.2
- net GNDIN: now also C21.2, C24.2, C25.2, JP10.2, JP9.1, U7.2, U7.3; no longer C16.2, C23.2, C27.2, JP6.2, JP8.1, U3.2, U3.3
- net GND_MIC1: now also JP3.1, U4.2, U4.3, U4.5; no longer JP1.1, U$2.2, U$2.3, U$2.5
- net GND_MIC3: now also U5.2, U5.3, U5.5; no longer U$14.2, U$14.3, U$14.5
- net MISO: now also JP7.3, U6.18; no longer SDCARD.3, U1.18
- net MOSI: now also JP7.4, U6.17; no longer SDCARD.4, U1.17
- net N$1: now also C5.1, R6.P$2, R7.P$1, U3.3; no longer C2.1, IC1.3, R3.P$2, R4.P$1
- net N$10: now also C10.2, R18.P$1, U3.13; no longer C8.2, IC1.13, R20.P$1
- net N$12: now also C2.1, JP2.3; no longer C3.1, JP3.3
- net N$13: now also C4.2, R1.P$1, U2.1; no longer C21.2, R2.P$1, U$1.1
- net N$14: now also C17.1, JP6.6; no longer C15.1, PRG.6
- net N$15: now also JP3.2, U4.4; no longer JP1.2, U$2.4
- net N$16: now also JP3.3, U4.1; no longer JP1.3, U$2.1
- net N$17: now also C18.2, U6.9; no longer C1.2, U1.9
- net N$18: now also C19.2, U6.10; no longer C5.2, U1.10
- net N$19: now also JP7.1; no longer SDCARD.1
- net N$2: now also C2.2, R2.P$1, U3.5; no longer C3.2, IC1.5, R12.P$1
- net N$20: now also C20.1, R25.P$2, U6.20, U6.21; no longer C13.1, R30.P$2, U1.20, U1.21
- net N$21: now also U5.4; no longer U$14.4
- net N$22: now also R29.P$1; no longer R10.P$1
- net N$23: now also R26.P$1; no longer R6.P$1
- net N$24: now also R27.P$1; no longer R7.P$1
- net N$25: now also R28.P$1; no longer R8.P$1
- net N$27: now also C24.1, U7.4; no longer C27.1, U3.4
- net N$28: now also IC1.2, R13.P$2, R15.P$1; no longer IC2.2, R23.P$2, R24.P$1
- net N$29: now also U5.1; no longer U$14.1
- net N$3: now also R3.P$1, R8.P$1, U3.6; no longer IC1.6, R13.P$1, R18.P$1
- net N$30: now also IC1.1; no longer IC2.1
- net N$31: now also IC1.5, R20.P$2, R22.P$2; no longer IC2.5, R25.P$2, R26.P$2
- net N$32: now also C12.2, R15.P$2, R20.P$1; no longer C17.2, R24.P$2, R25.P$1
- net N$33: now also IC1.6, R19.P$2, R23.P$1; no longer IC2.6, R27.P$2, R28.P$1
- net N$34: now also JP11.1; no longer JP7.1
- net N$35: now also C22.1; no longer C24.1
- net N$4: now also C7.1, R8.P$2, U3.7; no longer C6.1, IC1.7, R18.P$2
- net N$5: now also C7.2, R9.P$1, U3.10; no longer C6.2, IC1.10, R14.P$1
- net N$6: now also C9.1, R12.P$2, U3.8; no longer C7.1, IC1.8, R19.P$2
- net N$7: now also R11.P$1, R12.P$1, U3.9; no longer IC1.9, R15.P$1, R19.P$1
- net N$8: now also C10.1, C11.1, C9.2; no longer C7.2, C8.1, C9.1
- net N$9: now also U3.12; no longer IC1.12
- net RESET: now also C17.2, R30.P$1, U6.1; no longer C15.2, R11.P$1, U1.1
- net RX: now also JP6.4, U6.2; no longer PRG.4, U1.2
- net SCK: now also JP7.5, U6.19; no longer SDCARD.5, U1.19
- net SCL: now also JP5.4, U6.28; no longer RTC.4, U1.28
- net SDA: now also JP5.3, U6.27; no longer RTC.3, U1.27
- net TX: now also JP6.5, U6.3; no longer PRG.5, U1.3
- net VBATT: now also C23.1, JP8.2; no longer C25.1, JP5.2
- net VCC: now also C1.1, C15.1, C3.1, C6.1, IC1.8, JP1.2, JP2.4, R10.1, R4.P$1, R6.P$1, U1.1, U2.5, U3.4; no longer C10.1, C11.1, C18.1, C4.1, IC1.4, IC2.8, JP2.2, JP3.4, R1.P$1, R21.1, R3.P$1, U$1.5, U2.1
- net VDD: now also C16.1, JP5.2, JP6.3, JP7.2, R25.P$1, R30.P$2, U6.7; no longer C14.1, PRG.3, R11.P$2, R30.P$1, RTC.2, SDCARD.2, U1.7
- net VGND: now also C13.1, C8.1, IC1.3, JP2.2, R1.P$2, R11.P$2, R19.P$1, R2.P$2, R3.P$2, R9.P$2, U3.1, U3.2; no longer C12.1, C20.1, IC1.1, IC1.2, IC2.3, JP3.2, R12.P$2, R13.P$2, R14.P$2, R15.P$2, R27.P$1, R5.P$2
- net VIN: now also C21.1, JP9.2, U7.1; no longer C23.1, JP8.2, U3.1
- net VOUT: now also C25.1, JP10.1, U7.5; no longer C16.1, JP6.1, U3.5
- net X1: now also IC1.7, R23.P$2, R24.P$1; no longer IC2.7, R28.P$2, R29.P$1
- net XXX: now also C11.2, R18.P$2, R21.P$1, U3.14; no longer C9.2, IC1.14, R20.P$2, R22.P$1
Routing:
- net VBATT: track 31.3 -> 30.3 mm
- net N$34: track 17.7 -> 17.1 mm
Other:
- board size 99.7 x 48.6 mm -> 100 x 48.6 mm
- board text added: "BatNode V0.21"
- board text removed: "BatNode V0.2"
