File: circuit/Eagle/BatNode/BatNode.sch (EAGLE design)
At the start: 90 parts, among them IC1 TL974, IC2 TL972, Q1 BC547, U1 ATMEGA328P_PDIP, U3 TPS79147

Commit message: BatNode v0.21
Parts:
- removed C27: 0.1u, SparkFun-Capacitors:1.0UF-25V-+80/-20(0805)
- removed IC2: TL972, SparkFun-AnalogIC:OPAMP-DUALU
- removed PRG, SDCARD: (no value), SparkFun-Connectors:M06LOCK
- removed RTC: (no value), SparkFun-Connectors:M04LOCK
- removed U$1: LMV331, BatNodeParts:LMV339
- added C19: 22p, SparkFun-Capacitors:CAPPTH
- added JP10, JP11: VOUT, SparkFun-Connectors:M02LOCK
- added JP9: VIN, SparkFun-Connectors:M02LOCK
- added U6: ATMEGA328P_PDIP, SparkFun-DigitalIC:ATMEGA328P_PDIP
- added U7: TPS79147, SparkFun-PowerIC:V_REG_LDOSMD
- C1: value 22p -> 100u; device SparkFun-Capacitors:CAPPTH -> SparkFun-Capacitors:CAP_POLPTH1
- C10: value 0.1u -> 680p; device SparkFun-Capacitors:1.0UF-25V-+80/-20(0805) -> resistor:C-EU025-030X050
- C11: value 0.1u -> 1n; device SparkFun-Capacitors:1.0UF-25V-+80/-20(0805) -> resistor:C-EU025-030X050
- C12: device SparkFun-Capacitors:1.0UF-25V-+80/-20(0805) -> resistor:C-EU025-030X050
- C13: value 100n -> 4.7n; device SparkFun-Passives:CAP0805 -> resistor:C-EU025-030X050
- C14: value 100n -> 10n; device SparkFun-Passives:CAP0805 -> resistor:C-EU025-030X050
- C15: value 100n -> 0.1u; device SparkFun-Passives:CAP0805 -> SparkFun-Capacitors:1.0UF-25V-+80/-20(0805)
- C16, C17: value 1u -> 100n; device resistor:C-EU025-030X050 -> SparkFun-Passives:CAP0805
- C18: value 0.1u -> 22p; device SparkFun-Capacitors:1.0UF-25V-+80/-20(0805) -> SparkFun-Capacitors:CAPPTH
- C2: value 1u -> 10n; device SparkFun-Capacitors:1.0UF-25V-+80/-20(0805) -> resistor:C-EU025-030X050
- C20: value 4.7n -> 100n; device resistor:C-EU025-030X050 -> SparkFun-Passives:CAP0805
- C21: value 10p -> 0.1u; device resistor:C-EU025-030X050 -> SparkFun-Capacitors:1.0UF-25V-+80/-20(0805)
- C22: value 10n -> 1u
- C23: value 0.1u -> 1u; device SparkFun-Capacitors:1.0UF-25V-+80/-20(0805) -> resistor:C-EU025-030X050
- C24: value 1u -> 0.1u; device resistor:C-EU025-030X050 -> SparkFun-Capacitors:1.0UF-25V-+80/-20(0805)
- C3, C6: value 10n -> 0.1u; device resistor:C-EU025-030X050 -> SparkFun-Capacitors:1.0UF-25V-+80/-20(0805)
- C4: value 100u -> 10p; device SparkFun-Capacitors:CAP_POLPTH1 -> resistor:C-EU025-030X050
- C5: value 22p -> 1u; device SparkFun-Capacitors:CAPPTH -> SparkFun-Capacitors:1.0UF-25V-+80/-20(0805)
- C7: value 1n -> 10n
- C8: value 680p -> 1u; device resistor:C-EU025-030X050 -> SparkFun-Capacitors:1.0UF-25V-+80/-20(0805)
- IC1: value TL974 -> TL972; device SparkFun-AnalogIC:LMV324 -> SparkFun-AnalogIC:OPAMP-DUALU
- JP1: value MIC -> PWR; device SparkFun-Connectors:M03LOCK -> SparkFun-Connectors:M02LOCK
- JP2: value PWR -> MIC; device SparkFun-Connectors:M02LOCK -> SparkFun-Connectors:M04PTH
- JP3: device SparkFun-Connectors:M04PTH -> SparkFun-Connectors:M03LOCK
- JP5: value BAT -> (none); device SparkFun-Connectors:M02LOCK -> SparkFun-Connectors:M04LOCK
- JP6, JP7: value VOUT -> (none); device SparkFun-Connectors:M02LOCK -> SparkFun-Connectors:M06LOCK
- JP8: value VIN -> BAT
- R1: value 4.7k -> 2.2k
- R10: value 2.2k -> PHOTOCELLPTH; device SparkFun-Resistors:RESISTORAXIAL-0.3 -> SparkFun-Sensors:PHOTOCELLPTH
- R11: value 10k -> 6.8k; device SparkFun-Resistors:RESISTORAXIAL-0.3 -> SparkFun-Passives:RESISTORAXIAL-0.3
- R12: value 1k -> 100k
- R13: value 6.8k -> 4.7k
- R14: value 1k -> 10k
- R15: value 6.8k -> 22k
- R18: value 100k -> 22k
- R19: value 100k -> 4.7k
- R2: value 1Meg -> 1k
- R20: value 22k -> 4.7k
- R21: value PHOTOCELLPTH -> 330; device SparkFun-Sensors:PHOTOCELLPTH -> SparkFun-Passives:RESISTORAXIAL-0.3
- R22: value 330 -> 22k
- R23: value 4.7k -> 22k
- R24: value 22k -> 1k
- R25: value 4.7k -> 10uH
- R26, R28: value 22k -> 220; device SparkFun-Passives:RESISTORAXIAL-0.3 -> SparkFun-Resistors:RESISTORAXIAL-0.3
- R27: value 4.7k -> 220; device SparkFun-Passives:RESISTORAXIAL-0.3 -> SparkFun-Resistors:RESISTORAXIAL-0.3
- R29: value 1k -> 2.2k; device SparkFun-Passives:RESISTORAXIAL-0.3 -> SparkFun-Resistors:RESISTORAXIAL-0.3
- R3: value 47k -> 6.8k
- R30: value 10uH -> 10k; device SparkFun-Passives:RESISTORAXIAL-0.3 -> SparkFun-Resistors:RESISTORAXIAL-0.3
- R4: value 47k -> 4.7k
- R5: value 2.2k -> 1Meg
- R6, R7: value 220 -> 47k; device SparkFun-Resistors:RESISTORAXIAL-0.3 -> SparkFun-Passives:RESISTORAXIAL-0.3
- R8: value 220 -> 100k; device SparkFun-Resistors:RESISTORAXIAL-0.3 -> SparkFun-Passives:RESISTORAXIAL-0.3
- R9: value 10k -> 1k
- U1: value ATMEGA328P_PDIP -> (none); device SparkFun-DigitalIC:ATMEGA328P_PDIP -> SparkFun-Sensors:TMP36GT9
- U2: value (none) -> LMV331; device SparkFun-Sensors:TMP36GT9 -> BatNodeParts:LMV339
- U3: value TPS79147 -> LMV324; device SparkFun-PowerIC:V_REG_LDOSMD -> SparkFun-AnalogIC:LMV324
- renumbered GND-CONNECT to X12, RST to S3, U$14 to U5, U$15 to U8, U$2 to U4, V-CONNECT to X11
Connections:
- net A0: now also C14.1, R24.2, U6.PC0(ADC0); no longer C22.1, R29.2, U1.PC0(ADC0)
- net A1: now also U1.VOUT, U6.PC1(ADC1); no longer U1.PC1(ADC1), U2.VOUT
- net A2: now also R10.P$2, R14.1, U6.PC2(ADC2); no longer R21.P$2, R9.1, U1.PC2(ADC2)
- net A3: now also U6.PC3(ADC3); no longer U1.PC3(ADC3)
- net AGND: now also C1.-, C12.1, C14.2, C15.2, C3.2, C5.2, C6.2, C8.2, IC1A.V-, JP1.1, R14.2, R22.1, R7.2, U1.GND, U2.V-, U3G1.-V; no longer C10.2, C11.2, C12.2, C17.1, C18.2, C2.2, C22.2, C4.-, IC1G1.-V, IC2A.V-, JP3.1, R26.1, R4.2, R9.2, U$1.V-, U2.GND
- net CS: now also JP7.6, U6.PB2(SS/OC1B); no longer SDCARD.6, U1.PB2(SS/OC1B)
- net D2: now also U6.PD2(INT0); no longer U1.PD2(INT0)
- net D3: now also R26.2, U6.PD3(INT1); no longer R6.2, U1.PD3(INT1)
- net D4: now also U6.PD4(XCK/T0); no longer U1.PD4(XCK/T0)
- net D5: now also C4.1, R4.2, R5.2, U2.OUT, U6.PD5(T1); no longer C21.1, R1.2, R2.2, U$1.OUT, U1.PD5(T1)
- net D6: now also R27.2, U6.PD6(AIN0); no longer R7.2, U1.PD6(AIN0)
- net D7: now also R29.2, U6.PD7(AIN1); no longer R10.2, U1.PD7(AIN1)
- net D8: now also U6.PB0(ICP); no longer U1.PB0(ICP)
- net D9: now also R28.2, U6.PB1(OC1A); no longer R8.2, U1.PB1(OC1A)
- net FILTER: now also C13.2, R13.1, R21.2, U2.-IN; no longer C20.2, R22.2, R23.1, U$1.-IN
- net GND: now also C16.2, C18.1, C19.1, C20.2, JP5.1, JP6.1, U6.GND@1, U6.GND@2; no longer C1.1, C13.2, C14.2, C5.1, PRG.1, RTC.1, U1.GND@1, U1.GND@2
- net GNDBATT: now also C22.2, C23.2, JP11.2, JP8.1; no longer C24.2, C25.2, JP5.1, JP7.2
- net GNDIN: now also C21.2, C24.2, C25.2, JP10.2, JP9.1, U7.EN, U7.GND; no longer C16.2, C23.2, C27.2, JP6.2, JP8.1, U3.EN, U3.GND
- net GND_MIC1: now also JP3.1; no longer JP1.1
- net MISO: now also JP7.3, U6.PB4(MISO); no longer SDCARD.3, U1.PB4(MISO)
- net MOSI: now also JP7.4, U6.PB3(MOSI/OC2); no longer SDCARD.4, U1.PB3(MOSI/OC2)
- net N$1: now also C5.1, R6.2, R7.1, U3G1.+IN; no longer C2.1, IC1G1.+IN, R3.2, R4.1
- net N$10: now also C10.2, R18.1, U3G4.-IN; no longer C8.2, IC1G4.-IN, R20.1
- net N$12: now also C2.1, JP2.3; no longer C3.1, JP3.3
- net N$13: now also C4.2, R1.1, U2.+IN; no longer C21.2, R2.1, U$1.+IN
- net N$14: now also C17.1, JP6.6; no longer C15.1, PRG.6
- net N$15: now also JP3.2; no longer JP1.2
- net N$16: now also JP3.3; no longer JP1.3
- net N$17: now also C18.2, U6.PB6(XTAL1/TOSC1); no longer C1.2, U1.PB6(XTAL1/TOSC1)
- net N$18: now also C19.2, U6.PB7(XTAL2/TOSC2); no longer C5.2, U1.PB7(XTAL2/TOSC2)
- net N$19: now also JP7.1; no longer SDCARD.1
- net N$2: now also C2.2, R2.1, U3G3.+IN; no longer C3.2, IC1G3.+IN, R12.1
- net N$20: now also C20.1, R25.2, U6.AREF, U6.AVCC; no longer C13.1, R30.2, U1.AREF, U1.AVCC
- net N$22: now also R29.1; no longer R10.1
- net N$23: now also R26.1; no longer R6.1
- net N$24: now also R27.1; no longer R7.1
- net N$25: now also R28.1; no longer R8.1
- net N$27: now also C24.1, U7.BP; no longer C27.1, U3.BP
- net N$28: now also IC1A.-IN, R13.2, R15.1; no longer IC2A.-IN, R23.2, R24.1
- net N$3: now also R3.1, R8.1, U3G3.-IN; no longer IC1G3.-IN, R13.1, R18.1
- net N$30: now also IC1A.OUT; no longer IC2A.OUT
- net N$31: now also IC1B.+IN, R20.2, R22.2; no longer IC2B.+IN, R25.2, R26.2
- net N$32: now also C12.2, R15.2, R20.1; no longer C17.2, R24.2, R25.1
- net N$33: now also IC1B.-IN, R19.2, R23.1; no longer IC2B.-IN, R27.2, R28.1
- net N$34: now also JP11.1; no longer JP7.1
- net N$35: now also C22.1; no longer C24.1
- net N$4: now also C7.1, R8.2, U3G3.OUT; no longer C6.1, IC1G3.OUT, R18.2
- net N$5: now also C7.2, R9.1, U3G2.+IN; no longer C6.2, IC1G2.+IN, R14.1
- net N$6: now also C9.1, R12.2, U3G2.OUT; no longer C7.1, IC1G2.OUT, R19.2
- net N$7: now also R11.1, R12.1, U3G2.-IN; no longer IC1G2.-IN, R15.1, R19.1
- net N$8: now also C10.1, C11.1, C9.2; no longer C7.2, C8.1, C9.1
- net N$9: now also U3G4.+IN; no longer IC1G4.+IN
- net RESET: now also C17.2, R30.1, U6.PC6(/RESET); no longer C15.2, R11.1, U1.PC6(/RESET)
- net RX: now also JP6.4, U6.PD0(RXD); no longer PRG.4, U1.PD0(RXD)
- net SCK: now also JP7.5, U6.PB5(SCK); no longer SDCARD.5, U1.PB5(SCK)
- net SCL: now also JP5.4, U6.PC5(ADC5/SCL); no longer RTC.4, U1.PC5(ADC5/SCL)
- net SDA: now also JP5.3, U6.PC4(ADC4/SDA); no longer RTC.3, U1.PC4(ADC4/SDA)
- net TX: now also JP6.5, U6.PD1(TXD); no longer PRG.5, U1.PD1(TXD)
- net VBATT: now also C23.1, JP8.2; no longer C25.1, JP5.2
- net VCC: now also C1.+, C15.1, C3.1, C6.1, IC1A.V+, JP1.2, JP2.4, R10.P$1, R4.1, R6.1, U1.VCC, U2.V+, U3G1.+V; no longer C10.1, C11.1, C18.1, C4.+, IC1G1.+V, IC2A.V+, JP2.2, JP3.4, R1.1, R21.P$1, R3.1, U$1.V+, U2.VCC
- net VDD: now also C16.1, JP5.2, JP6.3, JP7.2, R25.1, R30.2, U6.VCC; no longer C14.1, PRG.3, R11.2, R30.1, RTC.2, SDCARD.2, U1.VCC
- net VGND: now also C13.1, C8.1, IC1A.+IN, JP2.2, R1.2, R11.2, R19.1, R2.2, R3.2, R9.2, U3G1.-IN, U3G1.OUT; no longer C12.1, C20.1, IC1G1.-IN, IC1G1.OUT, IC2A.+IN, JP3.2, R12.2, R13.2, R14.2, R15.2, R27.1, R5.2
- net VIN: now also C21.1, JP9.2, U7.IN; no longer C23.1, JP8.2, U3.IN
- net VOUT: now also C25.1, JP10.1, U7.OUT; no longer C16.1, JP6.1, U3.OUT
- net X1: now also IC1B.OUT, R23.2, R24.1; no longer IC2B.OUT, R28.2, R29.1
- net XXX: now also C11.2, R18.2, R21.1, U3G4.OUT; no longer C9.2, IC1G4.OUT, R20.2, R22.1
Other:
- moved on the sheet: C10, C11, C12, C13, C14, C15, C16, C17, C18, C2, C20, C21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
